File: Eagle/Qwiic_Iridium_9603N.sch (EAGLE design)
At the start: 59 parts, among them J1 IRIDIUM_9603N, J3 PTH, J6 ISP, J7 U.FL, Q2 5.8A/30V/35mΩ, U1 ATTINY841SOIC, U2 LTC3225EDDB#TRMPBF, U3 ADM4210-1

Commit message: Updated the SMD standoffs
Updated the Iridium 9603N and the SMD standoffs. The standoffs will now appear in the BOM.
Updated the PROD_IDs for the New_Parts.
The component positions should all be exactly the same, so no need to update the production panel.
Parts:
- added J10, J9: STANDOFFS_M2X0.4_STEEL_6MM, New_Parts:STANDOFFS_M2X0.4_STEEL_6MM
- C5, C6: device SparkFun-Capacitors:1F-2.7V(PTH)CPOL-RADIAL-1H-2.7V -> New_Parts:1F-2.7V(PTH)CPOL-RADIAL-1H-2.7V
- J1: device Qwiic_Iridium_9603N:IRIDIUM_9603N -> New_Parts:IRIDIUM_9603N
- R1, R12: device Qwiic_Iridium_9603N:1KOHM-0603-1/10W-1% -> SparkFun-Resistors:1KOHM-0603-1/10W-1%
- R9: value 0.012 Ohm -> 0.012R; device SparkFun-Resistors:RESISTOR0603 -> New_Parts:RESISTOR_0603_12MILLIOHM0603
- U1: device Qwiic_Iridium_9603N:ATTINY841SOIC -> New_Parts:ATTINY841SOIC
- U2: device Qwiic_Iridium_9603N:LTC3225EDDB-TRMPBFDFN300X200-10L -> New_Parts:LTC3225EDDB-TRMPBFDFN300X200-10L
- U3: device Qwiic_Iridium_9603N:ADM4210-1 -> New_Parts:ADM4210-1
Connections:
- net GND: now also J10.1, J9.1; no longer J1.HOLE1, J1.HOLE2
